File: AsksinPP_developments/PCBs/HB-UNI-SEN-BATT_FUEL4EP/HB-UNI-SEN-BATT_FUEL4EP.sch (KiCad schematic (older format))
At the start: 24 parts, among them J1 Conn_01x02, J10 BAT, J2 Conn_01x02, J3 Conn_01x02, J4 Conn_01x02, J5 ISP Programmer, J6 Conn_01x04, J7 Conn_01x04, J8 Conn_01x04, J9 Conn_01x04, Q1 IRLU024N, SW1 config button

Commit message: added pre-release of HB-UNI-SEN-BATT_FUEL4EP (still under test!)
Parts:
- removed AE1: 8.6 cm isolated wire antenna, symbol Device:Antenna
- added JP2: cut for accus, Jumper:SolderJumper-2_P1.3mm_Bridged_Pad1.0x1.5mm, symbol Jumper:SolderJumper_2_Bridged
- BT1, BT2: footprint Homebrew:BATTERY_HOLDER_GOOBAY_AA -> FUEL4EP:BATTERY_HOLDER_GOOBAY_AA
- C1: footprint Capacitors_THT:CP_Radial_D4.0mm_P1.50mm -> Capacitor_THT:CP_Radial_D4.0mm_P1.50mm
- D1: footprint LEDs:LED_D3.0mm -> LED_THT:LED_D3.0mm
- J1, J2, J3, J4: footprint (none) -> Connector_PinHeader_2.54mm:PinHeader_1x02_P2.54mm_Vertical
- J10: value BAT -> charge; footprint (none) -> Connector_PinHeader_2.54mm:PinHeader_1x02_P2.54mm_Vertical
- J5: footprint (none) -> Connector_PinHeader_2.54mm:PinHeader_1x06_P2.54mm_Vertical
- J6, J7, J8, J9: footprint (none) -> Connector_PinHeader_2.54mm:PinHeader_1x04_P2.54mm_Vertical
- JP1: value SolderJumper_2_Open -> NO; footprint (none) -> FUEL4EP:SolderJumper-2_P1.3mm_Open_Pad1.0x1.5mm
- Module1: value CC1101_transceiver_module -> CC1101; footprint (none) -> FUEL4EP:CC1101
- Module2: footprint (none) -> FUEL4EP:Tindie_ArduinoProMiniXL_1284P_V2
- Q1: footprint TO_SOT_Packages_THT:TO-251_IPAK_Vertical -> Package_TO_SOT_THT:TO-251-3_Vertical
- R1, R3, R4, R5: footprint Resistors_THT:R_Axial_DIN0207_L6.3mm_D2.5mm_P2.54mm_Vertical -> Resistor_THT:R_Axial_DIN0207_L6.3mm_D2.5mm_P2.54mm_Vertical
- SW1: footprint (none) -> Button_Switch_THT:SW_PUSH_6mm_H5mm
Connections:
- net labels added: minusBAT, plusBAT
- wire segments 116 -> 108
- no-connect marks 21 -> 23
Other:
- note added: "alternatively an Arduino Pro Mini\ncan be used, too."
- note added: "connect an\n8.6 cm long isolated wire\nas antenna"
- moved on the sheet: C1, D1, JP1, Module2, R1, SW1

Commit message: PCBs/HB-UNI-SEN-BATT_FUEL4EP updates, now with gerber data for JLCPCB (not yet vaalidated by prototype!)
Parts:
- added H1, H2, H3, H4: MountingHole, FUEL4EP:MountingHole_2.2mm_M2_Pad_Via, symbol Mechanical:MountingHole
- added LOGO1: Logo_Open_Hardware_Small, FUEL4EP:CC-BY-ND-SA, symbol Graphic:Logo_Open_Hardware_Small
Connections:
- wire segments 108 -> 112
Changed lines of the file:
@@
 Text Notes 3600 5500 0    60   ~ 0
 alternatively an Arduino Pro Mini\ncan be used, too.
+$Comp
+L Mechanical:MountingHole H2
+U 1 1 615CD389
+P 9850 6050
+F 0 "H2" H 9950 6096 50  0000 L CNN
+F 1 "MountingHole" H 9950 6005 50  0000 L CNN
+F 2 "FUEL4EP:MountingHole_2.2mm_M2_Pad_Via" H 9850 6050 50  0001 C CNN
+F 3 "~" H 9850 6050 50  0001 C CNN
+	1    9850 6050
+	1    0    0    -1
+$EndComp
+$Comp
+L Mechanical:MountingHole H1
+U 1 1 615D61D1
+P 9850 5850
+F 0 "H1" H 9950 5896 50  0000 L CNN
+F 1 "MountingHole" H 9950 5805 50  0000 L CNN
+F 2 "FUEL4EP:MountingHole_2.2mm_M2_Pad_Via" H 9850 5850 50  0001 C CNN
+F 3 "~" H 9850 5850 50  0001 C CNN
+	1    9850 5850
+	1    0    0    -1
+$EndComp
+$Comp
+L Mechanical:MountingHole H3
+U 1 1 615EB334
+P 10550 5850
+F 0 "H3" H 10650 5896 50  0000 L CNN
+F 1 "MountingHole" H 10650 5805 50  0000 L CNN
+F 2 "FUEL4EP:MountingHole_2.2mm_M2_Pad_Via" H 10550 5850 50  0001 C CNN
+F 3 "~" H 10550 5850 50  0001 C CNN
+	1    10550 5850
+	1    0    0    -1
+$EndComp
+$Comp
+L Mechanical:MountingHole H4
+U 1 1 615F62AC
+P 10550 6050
+F 0 "H4" H 10650 6096 50  0000 L CNN
+F 1 "MountingHole" H 10650 6005 50  0000 L CNN
+F 2 "FUEL4EP:MountingHole_2.2mm_M2_Pad_Via" H 10550 6050 50  0001 C CNN
+F 3 "~" H 10550 6050 50  0001 C CNN
+	1    10550 6050
+	1    0    0    -1
+$EndComp
+$Comp
+L Graphic:Logo_Open_Hardware_Small LOGO1
+U 1 1 615DEE46
+P 10250 5400
+F 0 "LOGO1" H 10250 5675 50  0001 C CNN
+F 1 "Logo_Open_Hardware_Small" H 10250 5175 50  0001 C CNN
+F 2 "FUEL4EP:CC-BY-ND-SA" H 10250 5400 50  0001 C CNN
+F 3 "~" H 10250 5400 50  0001 C CNN
+	1    10250 5400
+	1    0    0    -1
+$EndComp
+$Comp
+L power:GND #PWR?
+U 1 1 615DE0A0
+P 3250 6850
+F 0 "#PWR?" H 3250 6600 50  0001 C CNN
+F 1 "GND" H 3255 6677 50  0000 C CNN
+F 2 "" H 3250 6850 50  0001 C CNN
+F 3 "" H 3250 6850 50  0001 C CNN
+	1    3250 6850
+	1    0    0    -1
+$EndComp
+Wire Wire Line
+	3150 6500 3250 6500
+Wire Wire Line
+	3250 6500 3250 6700
+Wire Wire Line
+	3150 6700 3250 6700
+Connection ~ 3250 6700
+Wire Wire Line
+	3250 6700 3250 6850
 $EndSCHEMATC

Commit message: Updates of PCBs/HB-UNI-SEN-BATT_FUEL4EP and HB-UNI-SEN-BATT_E07-868MS10_FUEL4EP
Parts:
- BT1, BT2: footprint FUEL4EP:BATTERY_HOLDER_GOOBAY_AA -> FUEL4EP:BatteryHolder_Keystone_2460_1xAA
Connections:
- net labels added: conBAT
- wire segments 112 -> 114
Changed lines of the file:
@@
 F 0 "BT1" H 1450 1350 50  0000 L CNN
 F 1 "AA" H 1450 1250 50  0000 L CNN
-F 2 "FUEL4EP:BATTERY_HOLDER_GOOBAY_AA" V 1350 1310 50  0001 C CNN
+F 2 "FUEL4EP:BatteryHolder_Keystone_2460_1xAA" V 1350 1310 50  0001 C CNN
 F 3 "" V 1350 1310 50  0001 C CNN
 	1    1350 1250
@@
 F 0 "BT2" H 2100 1350 50  0000 L CNN
 F 1 "AA" H 2100 1250 50  0000 L CNN
-F 2 "FUEL4EP:BATTERY_HOLDER_GOOBAY_AA" V 2000 1310 50  0001 C CNN
+F 2 "FUEL4EP:BatteryHolder_Keystone_2460_1xAA" V 2000 1310 50  0001 C CNN
 F 3 "" V 2000 1310 50  0001 C CNN
 	1    2000 1250
@@
 	1350 1350 1350 1450
 Wire Wire Line
-	1350 1450 1700 1450
+	1350 1450 1525 1450
 Wire Wire Line
 	2000 1450 2100 1450
@@
 Wire Wire Line
 	3250 6700 3250 6850
+Text Label 1525 1525 3    60   ~ 0
+conBAT
+Wire Wire Line
+	1525 1525 1525 1450
+Connection ~ 1525 1450
+Wire Wire Line
+	1525 1450 1700 1450
 $EndSCHEMATC

Commit message: Update of PCBs / added PCBs/HB-UNI-SEN-BATT_ATMega1284P_E07-868MS10_FUEL4EP (all draft only, not yet validated)
Parts:
- J10: footprint Connector_PinHeader_2.54mm:PinHeader_1x02_P2.54mm_Vertical -> Connector_PinHeader_2.54mm:PinHeader_1x03_P2.54mm_Vertical; symbol Connector_Generic:Conn_01x02 -> Connector_Generic:Conn_01x03
Connections:
- wire segments 114 -> 116
Other:
- note added: "2x Keystone 2460\nbattery holders"
Changed lines of the file:
@@
 	1350 950  2100 950
-Wire Wire Line
-	2400 950  2400 1150
 Wire Wire Line
 	2000 1350 2000 1450
@@
 	2800 1150 2800 1000
 $Comp
-L Connector_Generic:Conn_01x02 J10
+L Connector_Generic:Conn_01x03 J10
 U 1 1 615781C9
 P 2600 1150
-F 0 "J10" H 2550 1300 50  0000 L CNN
+F 0 "J10" H 2525 1375 50  0000 L CNN
 F 1 "charge" H 2500 900 50  0000 L CNN
-F 2 "Connector_PinHeader_2.54mm:PinHeader_1x02_P2.54mm_Vertical" H 2600 1150 50  0001 C CNN
+F 2 "Connector_PinHeader_2.54mm:PinHeader_1x03_P2.54mm_Vertical" H 2600 1150 50  0001 C CNN
 F 3 "~" H 2600 1150 50  0001 C CNN
 	1    2600 1150
@@
 Wire Wire Line
 	2400 1150 2800 1150
-Connection ~ 2400 1150
 Wire Wire Line
 	2000 6300 2000 6050
@@
 NoConn ~ 2000 6800
 NoConn ~ 750  4550
-Text Label 2100 850  0    60   ~ 0
+Text Label 2100 850  2    60   ~ 0
 plusBAT
 Wire Wire Line
 	2100 850  2100 950
-Connection ~ 2100 950
-Wire Wire Line
-	2100 950  2400 950
 Text Notes 3600 5500 0    60   ~ 0
 alternatively an Arduino Pro Mini\ncan be used, too.
@@
 $EndComp
 $Comp
-L power:GND #PWR?
+L power:GND #PWR0107
 U 1 1 615DE0A0
 P 3250 6850
-F 0 "#PWR?" H 3250 6600 50  0001 C CNN
+F 0 "#PWR0107" H 3250 6600 50  0001 C CNN
 F 1 "GND" H 3255 6677 50  0000 C CNN
 F 2 "" H 3250 6850 50  0001 C CNN
@@
 Wire Wire Line
 	1525 1450 1700 1450
+Wire Wire Line
+	2400 1150 2275 1150
+Wire Wire Line
+	2275 1150 2275 950
+Wire Wire Line
+	2275 950  2100 950
+Connection ~ 2400 1150
+Connection ~ 2100 950
+$Comp
+L power:VCC #PWR0109
+U 1 1 616B7371
+P 2400 1000
+F 0 "#PWR0109" H 2400 850 50  0001 C CNN
+F 1 "VCC" H 2415 1173 50  0000 C CNN
+F 2 "" H 2400 1000 50  0001 C CNN
+F 3 "" H 2400 1000 50  0001 C CNN
+	1    2400 1000
+	1    0    0    -1
+$EndComp
+Wire Wire Line
+	2400 1000 2400 1050
+Text Notes 600  825  0    60   ~ 0
+2x Keystone 2460\nbattery holders
 $EndSCHEMATC
