File: AsksinPP_developments/PCBs/HB_Pro_Mini_ATMEGA1284P_FUEL4EP/HB_Pro_Mini_ATMEGA1284P_FUEL4EP.kicad_sch (KiCad schematic)
At the start: 22 parts, among them J1 FTDI Basic, J2 Conn_01x12, J3 Conn_01x12, J4 Conn_01x05, J5 Conn_01x02, U1 ATMEGA1284P-MUR, U2 TPS61221DCK, Y2 8MHz

Commit message: PCBs/HB_Pro_Mini_ATMEGA1284P_FUEL4EP and PCBs/I2C_Module_SHT45_BME280_small_FUEL4EP: updates based of prototype ordering at JLCPCB
Parts:
- C1, C4, C6, C7, C8: LCSC C28233 -> C1525
- C5: LCSC C76991 -> C15525
- R1: LCSC C17414 -> C25744
Changed lines of the file:
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@@
 			)
 		)
-		(property "LCSC" "C28233"
+		(property "LCSC" "C1525"
 			(at 52.07 43.18 0)
 			(effects
@@
 			)
 		)
-		(property "LCSC" "C28233"
+		(property "LCSC" "C1525"
 			(at 92.71 161.29 0)
 			(effects
@@
 			)
 		)
-		(property "LCSC" "C28233"
+		(property "LCSC" "C1525"
 			(at 77.47 43.18 0)
 			(effects
@@
 			)
 		)
-		(property "LCSC" "C17414"
+		(property "LCSC" "C25744"
 			(at 62.23 38.1 0)
 			(effects
@@
 			)
 		)
-		(property "LCSC" "C28233"
+		(property "LCSC" "C1525"
 			(at 101.6 50.8 0)
 			(effects
@@
 			)
 		)
-		(property "LCSC" "C28233"
+		(property "LCSC" "C1525"
 			(at 52.07 80.01 0)
 			(effects
@@
 			)
 		)
-		(property "LCSC" "C76991"
+		(property "LCSC" "C15525"
 			(at 69.85 43.18 0)
 			(effects

Commit message: PCBs/HB_Pro_Mini_ATMEGA1284P_FUEL4EP: update of LCSC data for JLCPCB prototype production
Parts:
- R2: LCSC C23345 -> C25092; TYPE 0603 -> 0402
Changed lines of the file:
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@@
 			)
 		)
-		(property "TYPE" "0603"
+		(property "TYPE" "0402"
 			(at 86.36 45.72 0)
 			(effects
@@
 			)
 		)
-		(property "LCSC" "C23345"
+		(property "LCSC" "C25092"
 			(at 86.36 45.72 0)
 			(effects
